File: Untitled/Untitled.kicad_sch (KiCad schematic)
At the start: 0 parts

Commit message: Started PCB work
Parts:
- added J1, J2, J3: USB_C_Receptacle, symbol Connector:USB_C_Receptacle
- added P1, P2: USB_C_Plug, symbol Connector:USB_C_Plug
Connections:
- new net: J1.A1 (GND), J1.A12 (GND), J1.B1 (GND), J1.B12 (GND)
- new net: J1.A4 (VBUS), J1.A9 (VBUS), J1.B4 (VBUS), J1.B9 (VBUS)
- new net: J2.A1 (GND), J2.A12 (GND), J2.B1 (GND), J2.B12 (GND)
- new net: J2.A4 (VBUS), J2.A9 (VBUS), J2.B4 (VBUS), J2.B9 (VBUS)
- new net: P1.A1 (GND), P1.A12 (GND), P1.B1 (GND), P1.B12 (GND)
- new net: P1.A4 (VBUS), P1.A9 (VBUS), P1.B4 (VBUS), P1.B9 (VBUS)
- new net: P2.A1 (GND), P2.A12 (GND), P2.B1 (GND), P2.B12 (GND)
- new net: P2.A4 (VBUS), P2.A9 (VBUS), P2.B4 (VBUS), P2.B9 (VBUS)
- new net: J3.A1 (GND), J3.A12 (GND), J3.B1 (GND), J3.B12 (GND)
- new net: J3.A4 (VBUS), J3.A9 (VBUS), J3.B4 (VBUS), J3.B9 (VBUS)
